File: Hardware/DianeHAT/DianeHAT.kicad_sch (KiCad schematic)
At the start: 0 parts

Commit message: Set up symbols and started schematic
Parts:
- added U1: RASPBERRY_PI_ZERO_2_W, RASPBERRY_PI_ZERO_2_W:MODULE_RASPBERRY_PI_ZERO_2_W, symbol RASPBERRY_PI_ZERO_2_W:RASPBERRY_PI_ZERO_2_W
- added U2: ~, symbol INMP441:INMP441
Connections:
- new net: U1.38 (GPIO20), U2.3 (SD)
- new net: U1.12 (GPIO18/GPIO_GEN1), U2.4 (SCK)
- new net: U1.35 (GPIO19), U2.5 (WS)
- new net +3.3V: U2.2 (VDD)
- new net Earth: U1.14 (GND_14), U1.20 (GND_20), U1.25 (GND_25), U1.30 (GND_30), U1.34 (GND_34), U1.39 (GND_39), U1.6 (GND_6), U1.9 (GND_9), U2.1 (GND)
- no-connect marks 0 -> 1

Commit message: Update DianeHAT.kicad_sch
Parts:
- U2: value ~ -> INMP441
Changed lines of the file:
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@@
 			)
 		)
-		(property "Value" "~"
+		(property "Value" "INMP441"
 			(at 158.75 76.2 0)
 			(effects
